File: eagle/inkubator/control.brd (EAGLE design)
At the start: 100 x 80 mm, 29 parts, among them IC1 MEGA16-P, Q2 BS250, X1 USBPTH

Commit message: schematic finished, board part 1
Parts:
- removed JP1: (no value), pinhead:1X06
- removed JP2: (no value), pinhead:1X05
- added C10, C11: 4u7, resistor:E5-5
- added C12, C13, C8, C9: 100n, resistor:C025-025X050
- added C6, C7: 10u, resistor:E2,5-5
- added H1, H2, H3, H4: MOUNT-HOLE3.2, holes:3,2
- added ISP: (no value), pinhead:2X03
- added PELT, PWR_PELT: (no value), con-wago-508:W237-132
- added Q3, Q4, Q5, Q6: IRF530, transistor-power:TO220BV
- R7, R9: device resistor:R0805 -> resistor:0207/10
- moved D1 143.7 mm to (85.1, 16.5), turned to 270 degrees
- moved U$2 142.7 mm to (47.6, 57.1)
- moved R2 130.2 mm to (90.2, 62.9), turned to 180 degrees
- moved R8 129.4 mm to (80.0, 26.7), turned to 180 degrees
- moved R9 124.7 mm to (80.0, 33.0), turned to 180 degrees
- moved U$1 123.9 mm to (35.6, 57.1)
- moved R4 123.2 mm to (62.2, 8.26), turned to 180 degrees
- moved LCD 120.4 mm to (76.2, 54.0), turned to 180 degrees
- moved R7 120.3 mm to (80.0, 29.2), turned to 180 degrees
- moved C5 117.4 mm to (47.0, 19.1)
- moved C1 113.3 mm to (48.3, 16.5)
- moved D2 110.3 mm to (90.2, 16.5), turned to 270 degrees
- moved RST 108.6 mm to (41.9, 16.5)
- moved C3 108.5 mm to (41.9, 12.7)
- moved X1 106.7 mm to (90.2, 27.9), turned to 180 degrees
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Connections:
- new net MISO: IC1.7, ISP.1
- new net MOSI: IC1.6, ISP.4
- new net N$41: Q5.G, U$2.3
- new net N$42: Q6.G, U$2.8
- new net N$46: C10.+, C11.+, C12.1, C13.1, PWR_PELT.2, Q3.D, Q5.D
- new net RESET: C3.2, IC1.9, ISP.5, R1.1, RST.2
- new net SCK: IC1.8, ISP.3
- net +5V: now also C6.+, C7.+, ISP.2, U$1.1, U$2.1
- net GND: now also C10.-, C11.-, C12.2, C13.2, C6.-, C7.-, ISP.6, PWR_PELT.1, Q4.S, Q6.S, U$1.7, U$2.7
- net N$3: now also IC1.33, U$2.5; no longer C3.2, IC1.9, R1.1, RST.2
- net N$30: now also IC1.34, U$2.6; no longer IC1.37, JP2.5
- net N$31: now also IC1.35, U$1.5; no longer IC1.36, JP2.4
- net N$32: now also IC1.36, U$1.6; no longer IC1.35, JP2.3
- net N$33: now also C9.1, U$1.2; no longer IC1.34, JP2.2
- net N$34: now also C8.1, U$2.2; no longer IC1.33, JP2.1
- net N$35: now also C8.2, U$2.4; no longer IC1.3, JP1.6
- net N$36: now also C9.2, U$1.4; no longer IC1.4, JP1.5
- net N$37: now also PELT.1, Q3.S, Q4.D; no longer IC1.5, JP1.4
- net N$38: now also PELT.2, Q5.S, Q6.D; no longer IC1.6, JP1.3
- net N$39: now also Q3.G, U$1.3; no longer IC1.7, JP1.2
- net N$40: now also Q4.G, U$1.8; no longer IC1.8, JP1.1
Routing:
- net +5V: track 0.00 -> 165.5 mm
- net RESET: track 0.00 -> 37.0 mm
- net N$21: track 0.00 -> 29.7 mm, vias 0 -> 2
- net N$7: track 0.00 -> 25.8 mm
- net N$8: track 0.00 -> 25.4 mm
- net N$9: track 0.00 -> 24.3 mm
- net N$10: track 0.00 -> 24.3 mm
- net N$11: track 0.00 -> 23.6 mm
- net N$12: track 0.00 -> 23.2 mm
- net N$13: track 0.00 -> 22.8 mm
- net N$14: track 0.00 -> 22.1 mm
- net N$29: track 0.00 -> 18.1 mm
- net N$18: track 0.00 -> 18.1 mm
- net N$25: track 0.00 -> 16.9 mm
- net N$4: track 0.00 -> 16.3 mm
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- added copper zone on layer 16, net GND

Commit message: board - almost done
Parts:
- moved Q4 51.8 mm to (12.7, 50.8), turned to 90 degrees
- moved Q3 36.4 mm to (12.7, 62.2), turned to 90 degrees
- moved Q6 34.3 mm to (45.7, 77.5)
- moved C10 30.9 mm to (21.6, 59.7), turned to 270 degrees
- moved C13 24.8 mm to (26.0, 63.5), turned to 90 degrees
- moved C12 15.3 mm to (58.4, 65.4)
- moved C11 14.0 mm to (59.7, 69.8)
- moved R3 12.6 mm to (54.6, 55.2)
- moved Q5 11.4 mm to (57.1, 77.5)
- moved C9 11.1 mm to (31.1, 60.3)
- moved C8 9.94 mm to (43.8, 60.3)
- moved U$1 5.68 mm to (30.5, 54.6), flipped to the bottom, turned to 180 degrees
- moved C6 5.12 mm to (24.8, 54.6), turned to 270 degrees
- moved U$2 5.12 mm to (43.2, 54.6), flipped to the bottom, turned to 180 degrees
- moved C7 4.07 mm to (38.1, 54.6), turned to 270 degrees
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Connections:
- net N$37: now also PELT.2; no longer PELT.1
- net N$38: now also PELT.1; no longer PELT.2
Routing:
- net +5V: track 165.5 -> 209.1 mm
- net N$37: track 0.00 -> 37.0 mm
- net N$38: track 0.00 -> 33.9 mm
- net N$42: track 0.00 -> 32.3 mm, vias 0 -> 2
- net N$41: track 0.00 -> 22.0 mm
- net N$39: track 0.00 -> 20.5 mm
- net N$46: track 0.00 -> 20.3 mm
- net N$30: track 0.00 -> 16.1 mm
- net N$3: track 0.00 -> 15.6 mm
- net N$31: track 0.00 -> 15.1 mm
- net N$40: track 0.00 -> 14.8 mm
- net N$32: track 0.00 -> 14.5 mm
- net N$6: track 0.00 -> 3.81 mm
- net N$36: track 0.00 -> 2.97 mm
- net N$35: track 0.00 -> 2.97 mm
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
Commit message: board v1.0a
Parts:
- added C14: 100n, resistor:C025-025X050
- added C15: 330n, resistor:C025-025X050
- added IC2: 7805TV, linear:TO220V
- added LCD2, LCD_PWR: (no value), pinhead:1X03
- added LED1: (no value), led:LED3MM
- added R10: 270R, resistor:0207/10
- LCD: device pinhead:1X16 -> pinhead:1X10
- moved LCD 7.62 mm to (68.6, 51.4)
- moved Q1 3.81 mm to (54.6, 11.4)
- moved C1 2.54 mm to (50.8, 16.5)
- moved C2 2.54 mm to (55.9, 16.5)
- moved C5 2.01 mm to (46.4, 17.1), turned to 90 degrees
- moved UART 1.27 mm to (61.0, 16.5)
Connections:
- new net N$43: LED1.A, R10.2
- net +5V: now also C14.1, IC2.3, LCD_PWR.2, LED1.K; no longer LCD.2
- net GND: now also C14.2, C15.2, IC2.2, LCD.10, LCD_PWR.1, R10.1; no longer LCD.1, LCD.16
- net N$10: now also LCD.4; no longer LCD.10
- net N$11: now also LCD.5; no longer LCD.11
- net N$12: now also LCD.6; no longer LCD.12
- net N$13: now also LCD.7; no longer LCD.13
- net N$14: now also LCD.8; no longer LCD.14
- net N$15: now also LCD2.3; no longer LCD.6
- net N$16: now also LCD2.2; no longer LCD.5
- net N$17: now also LCD2.1; no longer LCD.4
- net N$46: now also C15.1, IC2.1
- net N$5: now also LCD.9, R3.1; no longer LCD.3, R2.S
- net N$6: now also LCD_PWR.3, R2.S; no longer LCD.15, R3.1
- net N$7: now also LCD.1; no longer LCD.7
- net N$8: now also LCD.2; no longer LCD.8
- net N$9: now also LCD.3; no longer LCD.9
Routing:
- net N$46: track 20.3 -> 96.4 mm, vias 0 -> 2
- net +5V: track 209.1 -> 248.3 mm
- net N$17: track 0.00 -> 5.71 mm
- net N$16: track 0.00 -> 5.71 mm
- net N$15: track 0.00 -> 5.71 mm
- net N$43: track 0.00 -> 4.45 mm
- net N$2: track 12.4 -> 13.2 mm
- net N$27: track 7.40 -> 7.93 mm
- net N$26: track 7.40 -> 7.93 mm
Other:
- board text added: "brmlab"
- board text added: "design by nephirus"
- board text added: "hackerspace prague"
- board text added: "incubator v1.0a"
