File: eagle/inkubator/control.sch (EAGLE design)
At the start: 29 parts, among them IC1 MEGA16-P, Q2 BS250, X1 USBPTH

Commit message: schematic finished, board part 1
Parts:
- removed JP1: (no value), pinhead:PINHD-1X6
- removed JP2: (no value), pinhead:PINHD-1X5
- added C10, C11: 4u7, resistor:CPOL-EUE5-5
- added C12, C13, C8, C9: 100n, resistor:C-EU025-025X050
- added C6, C7: 10u, resistor:CPOL-EUE2.5-5
- added H1, H2, H3, H4: MOUNT-HOLE3.2, holes:MOUNT-HOLE3.2
- added ISP: (no value), pinhead:PINHD-2X3
- added PELT, PWR_PELT: (no value), con-wago-508:W237-02P
- added Q3, Q4, Q5, Q6: IRF530, transistor-power:IRF530
- R7, R9: device resistor:R-EU_R0805 -> resistor:R-EU_0207/10
Connections:
- new net MISO: IC1.(MISO)PB6, ISP.1
- new net MOSI: IC1.(MOSI)PB5, ISP.4
- new net N$41: Q5.G, U$2.HO
- new net N$42: Q6.G, U$2.LO
- new net N$46: C10.+, C11.+, C12.1, C13.1, PWR_PELT-2.KL, Q3.D, Q5.D
- new net RESET: C3.2, IC1.RESET, ISP.5, R1.1, RST.2
- new net SCK: IC1.(SCK)PB7, ISP.3
- net +5V: now also C6.+, C7.+, ISP.2, U$1.VDD, U$2.VDD
- net GND: now also C10.-, C11.-, C12.2, C13.2, C6.-, C7.-, ISP.6, PWR_PELT-1.KL, Q4.S, Q6.S, U$1.VSS, U$2.VSS
- net N$3: now also IC1.(ADC7)PA7, U$2.HI; no longer C3.2, IC1.RESET, R1.1, RST.2
- net N$30: now also IC1.(ADC6)PA6, U$2.LI; no longer IC1.(ADC3)PA3, JP2.5
- net N$31: now also IC1.(ADC5)PA5, U$1.HI; no longer IC1.(ADC4)PA4, JP2.4
- net N$32: now also IC1.(ADC4)PA4, U$1.LI; no longer IC1.(ADC5)PA5, JP2.3
- net N$33: now also C9.1, U$1.HB; no longer IC1.(ADC6)PA6, JP2.2
- net N$34: now also C8.1, U$2.HB; no longer IC1.(ADC7)PA7, JP2.1
- net N$35: now also C8.2, U$2.HS; no longer IC1.(AIN0/INT2)PB2, JP1.6
- net N$36: now also C9.2, U$1.HS; no longer IC1.(AIN1/OC0)PB3, JP1.5
- net N$37: now also PELT-1.KL, Q3.S, Q4.D; no longer IC1.(SS)PB4, JP1.4
- net N$38: now also PELT-2.KL, Q5.S, Q6.D; no longer IC1.(MOSI)PB5, JP1.3
- net N$39: now also Q3.G, U$1.HO; no longer IC1.(MISO)PB6, JP1.2
- net N$40: now also Q4.G, U$1.LO; no longer IC1.(SCK)PB7, JP1.1
Other:
- moved on the sheet: U$1, U$2

Commit message: board - almost done
Connections:
- net N$37: now also PELT-2.KL; no longer PELT-1.KL
- net N$38: now also PELT-1.KL; no longer PELT-2.KL
Other:
- moved on the sheet: PELT-1, PELT-2
Changed lines of the file:
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@@
 <instance part="Q5" gate="G$1" x="119.38" y="137.16" rot="MR0"/>
 <instance part="Q6" gate="G$1" x="119.38" y="104.14" rot="MR0"/>
-<instance part="PELT" gate="-1" x="99.06" y="116.84" rot="R90"/>
-<instance part="PELT" gate="-2" x="104.14" y="116.84" rot="R90"/>
+<instance part="PELT" gate="-1" x="106.68" y="116.84" rot="R90"/>
+<instance part="PELT" gate="-2" x="99.06" y="116.84" rot="R90"/>
 <instance part="PWR_PELT" gate="-1" x="101.6" y="167.64" rot="R270"/>
 <instance part="PWR_PELT" gate="-2" x="96.52" y="167.64" rot="R270"/>
@@
 <pinref part="Q4" gate="G$1" pin="D"/>
 <wire x1="83.82" y1="132.08" x2="83.82" y2="121.92" width="0.1524" layer="91"/>
-<pinref part="PELT" gate="-1" pin="KL"/>
+<pinref part="PELT" gate="-2" pin="KL"/>
 <wire x1="83.82" y1="121.92" x2="83.82" y2="109.22" width="0.1524" layer="91"/>
 <wire x1="99.06" y1="121.92" x2="83.82" y2="121.92" width="0.1524" layer="91"/>
@@
 <pinref part="Q6" gate="G$1" pin="D"/>
 <wire x1="116.84" y1="132.08" x2="116.84" y2="121.92" width="0.1524" layer="91"/>
-<pinref part="PELT" gate="-2" pin="KL"/>
+<pinref part="PELT" gate="-1" pin="KL"/>
 <wire x1="116.84" y1="121.92" x2="116.84" y2="109.22" width="0.1524" layer="91"/>
-<wire x1="104.14" y1="121.92" x2="116.84" y2="121.92" width="0.1524" layer="91"/>
+<wire x1="106.68" y1="121.92" x2="116.84" y2="121.92" width="0.1524" layer="91"/>
 <junction x="116.84" y="121.92"/>
 </segment>

Commit message: board v1.0a
Parts:
- added C14: 100n, resistor:C-EU025-025X050
- added C15: 330n, resistor:C-EU025-025X050
- added IC2: 7805TV, linear:7805TV
- added LCD2, LCD_PWR: (no value), pinhead:PINHD-1X3
- added LED1: (no value), led:LED3MM
- added R10: 270R, resistor:R-EU_0207/10
- LCD: device pinhead:PINHD-1X16 -> pinhead:PINHD-1X10
Connections:
- new net N$43: LED1.A, R10.2
- net +5V: now also C14.1, IC2.VO, LCD_PWR.2, LED1.C; no longer LCD.2
- net GND: now also C14.2, C15.2, IC2.GND, LCD.10, LCD_PWR.1, R10.1; no longer LCD.1, LCD.16
- net N$10: now also LCD.4; no longer LCD.10
- net N$11: now also LCD.5; no longer LCD.11
- net N$12: now also LCD.6; no longer LCD.12
- net N$13: now also LCD.7; no longer LCD.13
- net N$14: now also LCD.8; no longer LCD.14
- net N$15: now also LCD2.3; no longer LCD.6
- net N$16: now also LCD2.2; no longer LCD.5
- net N$17: now also LCD2.1; no longer LCD.4
- net N$46: now also C15.1, IC2.VI
- net N$5: now also LCD.9, R3.1; no longer LCD.3, R2.S
- net N$6: now also LCD_PWR.3, R2.S; no longer LCD.15, R3.1
- net N$7: now also LCD.1; no longer LCD.7
- net N$8: now also LCD.2; no longer LCD.8
- net N$9: now also LCD.3; no longer LCD.9
