File: eagle/inkubator/peltier_regulator.sch (EAGLE design)
At the start: 17 parts, among them Q1 IRF540, Q2 IRF540, Q3 IRF540, Q4 IRF540

Commit message: peltier regulator board
Parts:
- added JP2: (no value), pinhead:PINHD-1X2
- added PAD1, PAD2, PAD3, PAD4, PAD5: (no value), wirepad:2,54/1,0
- C3, C4: device resistor:CPOL-EUE5-10.5 -> resistor:C-EUC1206
- JP1: device pinhead:PINHD-1X6 -> pinhead:PINHD-1X4
Connections:
- new net GND: C1.-, C2.-, C5.2, C6.2, JP1.1, PAD3.P, PAD5.P, Q2.S, Q4.S, U$1.VSS, U$2.VSS
- new net N$1: C3.2, U$1.HS
- new net N$10: C4.2, U$2.HS
- new net N$11: R3.2, U$2.HO
- new net N$12: R4.2, U$2.LO
- new net N$13: JP2.1, U$2.LI
- new net N$14: JP2.2, U$2.HI
- new net N$15: PAD1.P, Q1.S, Q2.D
- new net N$16: PAD2.P, Q3.S, Q4.D
- new net N$2: Q1.G, R1.2
- new net N$3: R2.1, U$1.LO
- new net N$4: Q2.G, R2.2
- new net N$5: R1.1, U$1.HO
- new net N$6: JP1.2, U$1.LI
- new net N$7: JP1.3, U$1.HI
- new net N$8: Q4.G, R4.1
- new net N$9: Q3.G, R3.1
- new net VCC: C1.+, C2.+, C3.1, C4.1, C5.1, C6.1, JP1.4, U$1.HB, U$1.VDD, U$2.HB, U$2.VDD
- new net VDD: PAD4.P, Q1.D, Q3.D
Other:
- moved on the sheet: C1, C2, C5, C6, Q1, Q2, Q3, Q4, R1, R2, R3, R4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
